File: VL53L1X.kicad_sch (KiCad schematic)
At the start: 0 parts

Commit message: Fix paths
Parts:
- added IC1: VL53L1X, VL53L1X:VL53L1X, symbol VL53L1X:VL53L1X
Changed lines of the file:
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@@
-(kicad_sch (version 20200310) (host eeschema "unknown")
-(  page "A4")
-  (symbol_instances)
+(kicad_sch (version 20201015) (generator eeschema)
+  (paper "A4")
+  (symbol (lib_id "VL53L1X:VL53L1X") (at 129.54 92.71 0) (unit 1)
+    (in_bom yes) (on_board yes)
+    (property "Reference" "IC1" (id 0) (at 147.32 85.09 0))
+    (property "Value" "VL53L1X" (id 1) (at 147.32 87.63 0))
+    (property "Footprint" "VL53L1X:VL53L1X" (id 2) (at 161.29 90.17 0)
+      (effects (font (size 1.27 1.27)) (justify left) hide)
+    )
+    (property "Datasheet" "https://componentsearchengine.com/Datasheets/1/VL53L1X.pdf" (id 3) (at 161.29 92.71 0)
+      (effects (font (size 1.27 1.27)) (justify left) hide)
+    )
+    (property "Description" "Long distance ranging Time-of-Flight sen" (id 4) (at 161.29 95.25 0)
+      (effects (font (size 1.27 1.27)) (justify left) hide)
+    )
+    (property "Height" "1" (id 5) (at 161.29 97.79 0)
+      (effects (font (size 1.27 1.27)) (justify left) hide)
+    )
+    (property "Manufacturer_Name" "STMicroelectronics" (id 6) (at 161.29 100.33 0)
+      (effects (font (size 1.27 1.27)) (justify left) hide)
+    )
+    (property "Manufacturer_Part_Number" "VL53L1X" (id 7) (at 161.29 102.87 0)
+      (effects (font (size 1.27 1.27)) (justify left) hide)
+    )
+  )
+  (sheet_instances
+    (path "/" (page "1"))
+  )
+  (symbol_instances
+    (path "/f0cffca8-9dbc-484e-8acc-15e3e8cbcb54"
+      (reference "IC1") (unit 1) (value "VL53L1X") (footprint "VL53L1X:VL53L1X")
+    )
+  )
 )
