File: VL53L1X.kicad_sch (KiCad schematic)
At the start: 1 part, among them IC1 VL53L1X

Commit message: schematic, layout, routing, all done.
Parts:
- added C1: 100 nF, Capacitor_SMD:C_0201_0603Metric_Pad0.64x0.40mm_HandSolder, symbol Device:C
- added C2: 4.7 uF, Capacitor_SMD:C_0201_0603Metric_Pad0.64x0.40mm_HandSolder, symbol Device:C
- added J1: Conn_01x06, Connector_JST:JST_SH_SM06B-SRSS-TB_1x06-1MP_P1.00mm_Horizontal, symbol Connector_Generic:Conn_01x06
Connections:
- net AVDD: now reaches IC1.1 (AVDDVCSEL)
- net AVDD: now also IC1.11 (AVDD), C1.1, C2.1, J1.2 (Pin_2)
- net SCL: now reaches IC1.10 (SCL)
- net SCL: now also J1.4 (Pin_4)
- net GND: now reaches IC1.12 (GND4)
- net GND: now also IC1.2 (AVSSVCSEL), IC1.3 (GND), IC1.4 (GND2), IC1.6 (GND3), C1.2, C2.2, J1.1 (Pin_1)
- net XSHUT: now reaches IC1.5 (XSHUT)
- net XSHUT: now also J1.6 (Pin_6)
- net GPIO1: now reaches IC1.7 (GPIO1)
- net GPIO1: now also J1.5 (Pin_5)
- net SDA: now reaches IC1.9 (SDA)
- net SDA: now also J1.3 (Pin_3)
- no-connect marks 0 -> 1
Changed lines of the file:
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@@
 (kicad_sch (version 20201015) (generator eeschema)
   (paper "A4")
+  (junction (at 120.65 97.79) (diameter 0.9144) (color 0 0 0 0))
+  (junction (at 120.65 100.33) (diameter 0.9144) (color 0 0 0 0))
+  (junction (at 120.65 105.41) (diameter 0.9144) (color 0 0 0 0))
+  (junction (at 195.58 92.71) (diameter 0.9144) (color 0 0 0 0))
+  (junction (at 210.82 105.41) (diameter 0.9144) (color 0 0 0 0))
+  (no_connect (at 167.64 95.25))
+  (wire (pts (xy 86.36 92.71) (xy 88.9 92.71))
+    (stroke (width 0) (type solid) (color 0 0 0 0))
+  )
+  (wire (pts (xy 86.36 95.25) (xy 88.9 95.25))
+    (stroke (width 0) (type solid) (color 0 0 0 0))
+  )
+  (wire (pts (xy 86.36 97.79) (xy 88.9 97.79))
+    (stroke (width 0) (type solid) (color 0 0 0 0))
+  )
+  (wire (pts (xy 86.36 100.33) (xy 88.9 100.33))
+    (stroke (width 0) (type solid) (color 0 0 0 0))
+  )
+  (wire (pts (xy 86.36 102.87) (xy 88.9 102.87))
+    (stroke (width 0) (type solid) (color 0 0 0 0))
+  )
+  (wire (pts (xy 86.36 105.41) (xy 88.9 105.41))
+    (stroke (width 0) (type solid) (color 0 0 0 0))
+  )
+  (wire (pts (xy 120.65 95.25) (xy 120.65 97.79))
+    (stroke (width 0) (type solid) (color 0 0 0 0))
+  )
+  (wire (pts (xy 120.65 95.25) (xy 129.54 95.25))
+    (stroke (width 0) (type solid) (color 0 0 0 0))
+  )
+  (wire (pts (xy 120.65 97.79) (xy 120.65 100.33))
+    (stroke (width 0) (type solid) (color 0 0 0 0))
+  )
+  (wire (pts (xy 120.65 97.79) (xy 129.54 97.79))
+    (stroke (width 0) (type solid) (color 0 0 0 0))
+  )
+  (wire (pts (xy 120.65 100.33) (xy 120.65 105.41))
+    (stroke (width 0) (type solid) (color 0 0 0 0))
+  )
+  (wire (pts (xy 120.65 100.33) (xy 129.54 100.33))
+    (stroke (width 0) (type solid) (color 0 0 0 0))
+  )
+  (wire (pts (xy 120.65 105.41) (xy 120.65 107.95))
+    (stroke (width 0) (type solid) (color 0 0 0 0))
+  )
+  (wire (pts (xy 120.65 105.41) (xy 129.54 105.41))
+    (stroke (width 0) (type solid) (color 0 0 0 0))
+  )
+  (wire (pts (xy 127 92.71) (xy 129.54 92.71))
+    (stroke (width 0) (type solid) (color 0 0 0 0))
+  )
+  (wire (pts (xy 127 102.87) (xy 129.54 102.87))
+    (stroke (width 0) (type solid) (color 0 0 0 0))
+  )
+  (wire (pts (xy 165.1 92.71) (xy 170.18 92.71))
+    (stroke (width 0) (type solid) (color 0 0 0 0))
+  )
+  (wire (pts (xy 165.1 95.25) (xy 167.64 95.25))
+    (stroke (width 0) (type solid) (color 0 0 0 0))
+  )
+  (wire (pts (xy 165.1 97.79) (xy 170.18 97.79))
+    (stroke (width 0) (type solid) (color 0 0 0 0))
+  )
+  (wire (pts (xy 165.1 100.33) (xy 170.18 100.33))
+    (stroke (width 0) (type solid) (color 0 0 0 0))
+  )
+  (wire (pts (xy 165.1 102.87) (xy 170.18 102.87))
+    (stroke (width 0) (type solid) (color 0 0 0 0))
+  )
+  (wire (pts (xy 165.1 105.41) (xy 170.18 105.41))
+    (stroke (width 0) (type solid) (color 0 0 0 0))
+  )
+  (wire (pts (xy 170.18 105.41) (xy 170.18 107.95))
+    (stroke (width 0) (type solid) (color 0 0 0 0))
+  )
+  (wire (pts (xy 195.58 88.9) (xy 195.58 92.71))
+    (stroke (width 0) (type solid) (color 0 0 0 0))
+  )
+  (wire (pts (xy 195.58 92.71) (xy 195.58 95.25))
+    (stroke (width 0) (type solid) (color 0 0 0 0))
+  )
+  (wire (pts (xy 195.58 92.71) (xy 210.82 92.71))
+    (stroke (width 0) (type solid) (color 0 0 0 0))
+  )
+  (wire (pts (xy 195.58 102.87) (xy 195.58 105.41))
+    (stroke (width 0) (type solid) (color 0 0 0 0))
+  )
+  (wire (pts (xy 195.58 105.41) (xy 210.82 105.41))
+    (stroke (width 0) (type solid) (color 0 0 0 0))
+  )
+  (wire (pts (xy 210.82 92.71) (xy 210.82 95.25))
+    (stroke (width 0) (type solid) (color 0 0 0 0))
+  )
+  (wire (pts (xy 210.82 102.87) (xy 210.82 105.41))
+    (stroke (width 0) (type solid) (color 0 0 0 0))
+  )
+  (wire (pts (xy 210.82 105.41) (xy 210.82 107.95))
+    (stroke (width 0) (type solid) (color 0 0 0 0))
+  )
+  (label "GND" (at 86.36 92.71 180)
+    (effects (font (size 1 1)) (justify right bottom))
+  )
+  (label "AVDD" (at 86.36 95.25 180)
+    (effects (font (size 1 1)) (justify right bottom))
+  )
+  (label "SDA" (at 86.36 97.79 180)
+    (effects (font (size 1 1)) (justify right bottom))
+  )
+  (label "SCL" (at 86.36 100.33 180)
+    (effects (font (size 1 1)) (justify right bottom))
+  )
+  (label "GPIO1" (at 86.36 102.87 180)
+    (effects (font (size 1 1)) (justify right bottom))
+  )
+  (label "XSHUT" (at 86.36 105.41 180)
+    (effects (font (size 1 1)) (justify right bottom))
+  )
+  (label "AVDD" (at 127 92.71 180)
+    (effects (font (size 1 1)) (justify right bottom))
+  )
+  (label "XSHUT" (at 127 102.87 180)
+    (effects (font (size 1 1)) (justify right bottom))
+  )
+  (label "GPIO1" (at 170.18 92.71 0)
+    (effects (font (size 1 1)) (justify left bottom))
+  )
+  (label "SDA" (at 170.18 97.79 0)
+    (effects (font (size 1 1)) (justify left bottom))
+  )
+  (label "SCL" (at 170.18 100.33 0)
+    (effects (font (size 1 1)) (justify left bottom))
+  )
+  (label "AVDD" (at 170.18 102.87 0)
+    (effects (font (size 1 1)) (justify left bottom))
+  )
+  (label "AVDD" (at 195.58 88.9 180)
+    (effects (font (size 1 1)) (justify right bottom))
+  )
+  (symbol (lib_id "power:GND") (at 120.65 107.95 0) (unit 1)
+    (in_bom yes) (on_board yes)
+    (property "Reference" "#PWR0101" (id 0) (at 120.65 114.3 0)
+      (effects (font (size 1.27 1.27)) hide)
+    )
+    (property "Value" "GND" (id 1) (at 121.92 113.03 0))
+    (property "Footprint" "" (id 2) (at 120.65 107.95 0)
+      (effects (font (size 1.27 1.27)) hide)
+    )
+    (property "Datasheet" "" (id 3) (at 120.65 107.95 0)
+      (effects (font (size 1.27 1.27)) hide)
+    )
+  )
+  (symbol (lib_id "power:GND") (at 170.18 107.95 0) (unit 1)
+    (in_bom yes) (on_board yes)
+    (property "Reference" "#PWR0102" (id 0) (at 170.18 114.3 0)
+      (effects (font (size 1.27 1.27)) hide)
+    )
+    (property "Value" "GND" (id 1) (at 171.45 113.03 0))
+    (property "Footprint" "" (id 2) (at 170.18 107.95 0)
+      (effects (font (size 1.27 1.27)) hide)
+    )
+    (property "Datasheet" "" (id 3) (at 170.18 107.95 0)
+      (effects (font (size 1.27 1.27)) hide)
+    )
+  )
+  (symbol (lib_id "power:GND") (at 210.82 107.95 0) (unit 1)
+    (in_bom yes) (on_board yes)
+    (property "Reference" "#PWR0103" (id 0) (at 210.82 114.3 0)
+      (effects (font (size 1.27 1.27)) hide)
+    )
+    (property "Value" "GND" (id 1) (at 212.09 113.03 0))
+    (property "Footprint" "" (id 2) (at 210.82 107.95 0)
+      (effects (font (size 1.27 1.27)) hide)
+    )
+    (property "Datasheet" "" (id 3) (at 210.82 107.95 0)
+      (effects (font (size 1.27 1.27)) hide)
+    )
+  )
+  (symbol (lib_id "Device:C") (at 195.58 99.06 0) (unit 1)
+    (in_bom yes) (on_board yes)
+    (property "Reference" "C1" (id 0) (at 199.39 97.79 0)
+      (effects (font (size 1.27 1.27)) (justify left))
+    )
+    (property "Value" "100 nF" (id 1) (at 199.39 100.33 0)
+      (effects (font (size 1.27 1.27)) (justify left))
+    )
+    (property "Footprint" "Capacitor_SMD:C_0201_0603Metric_Pad0.64x0.40mm_HandSolder" (id 2) (at 196.5452 102.87 0)
+      (effects (font (size 1.27 1.27)) hide)
+    )
+    (property "Datasheet" "~" (id 3) (at 195.58 99.06 0)
+      (effects (font (size 1.27 1.27)) hide)
+    )
+  )
+  (symbol (lib_id "Device:C") (at 210.82 99.06 0) (unit 1)
+    (in_bom yes) (on_board yes)
+    (property "Reference" "C2" (id 0) (at 214.63 97.79 0)
+      (effects (font (size 1.27 1.27)) (justify left))
+    )
+    (property "Value" "4.7 uF" (id 1) (at 214.63 100.33 0)
+      (effects (font (size 1.27 1.27)) (justify left))
+    )
+    (property "Footprint" "Capacitor_SMD:C_0201_0603Metric_Pad0.64x0.40mm_HandSolder" (id 2) (at 211.7852 102.87 0)
+      (effects (font (size 1.27 1.27)) hide)
+    )
+    (property "Datasheet" "~" (id 3) (at 210.82 99.06 0)
+      (effects (font (size 1.27 1.27)) hide)
+    )
+  )
+  (symbol (lib_id "Connector_Generic:Conn_01x06") (at 93.98 97.79 0) (unit 1)
+    (in_bom yes) (on_board yes)
+    (property "Reference" "J1" (id 0) (at 96.52 99.06 0)
+      (effects (font (size 1.27 1.27)) (justify left))
+    )
+    (property "Value" "Conn_01x06" (id 1) (at 96.52 101.6 0)
+      (effects (font (size 1.27 1.27)) (justify left))
+    )
+    (property "Footprint" "Connector_JST:JST_SH_SM06B-SRSS-TB_1x06-1MP_P1.00mm_Horizontal" (id 2) (at 93.98 97.79 0)
+      (effects (font (size 1.27 1.27)) hide)
+    )
+    (property "Datasheet" "~" (id 3) (at 93.98 97.79 0)
+      (effects (font (size 1.27 1.27)) hide)
+    )
+  )
   (symbol (lib_id "VL53L1X:VL53L1X") (at 129.54 92.71 0) (unit 1)
     (in_bom yes) (on_board yes)
@@
   )
   (symbol_instances
+    (path "/cbedb9ea-c4dc-4736-a205-0ab1ad555047"
+      (reference "#PWR0101") (unit 1) (value "GND") (footprint "")
+    )
+    (path "/df60deaa-bec3-45d2-982f-536e2bf43923"
+      (reference "#PWR0102") (unit 1) (value "GND") (footprint "")
+    )
+    (path "/8885ce45-ac03-4734-af4b-4cb834f154cd"
+      (reference "#PWR0103") (unit 1) (value "GND") (footprint "")
+    )
+    (path "/2991d22b-3b67-454f-b9b4-2498d91e6dda"
+      (reference "C1") (unit 1) (value "100 nF") (footprint "Capacitor_SMD:C_0201_0603Metric_Pad0.64x0.40mm_HandSolder")
+    )
+    (path "/577390c4-391b-4887-ab92-1f61b9f89d45"
+      (reference "C2") (unit 1) (value "4.7 uF") (footprint "Capacitor_SMD:C_0201_0603Metric_Pad0.64x0.40mm_HandSolder")
+    )
     (path "/f0cffca8-9dbc-484e-8acc-15e3e8cbcb54"
       (reference "IC1") (unit 1) (value "VL53L1X") (footprint "VL53L1X:VL53L1X")
     )
-  )
+    (path "/30bdb6ef-84c1-4370-b57d-93597d142f33"
+      (reference "J1") (unit 1) (value "Conn_01x06") (footprint "Connector_JST:JST_SH_SM06B-SRSS-TB_1x06-1MP_P1.00mm_Horizontal")
+    )
+  )
