File: VL53L1X.kicad_pcb (KiCad board)
At the start: 2 copper layers, 1 part, among them IC1 VL53L1X

Commit message: schematic, layout, routing, all done.
Parts:
- added C1: 100 nF, Capacitor_SMD:C_0201_0603Metric_Pad0.64x0.40mm_HandSolder, F.Cu at (149.0, 89.3)
- added C2: 4.7 uF, Capacitor_SMD:C_0201_0603Metric_Pad0.64x0.40mm_HandSolder, F.Cu at (149.0, 88.5)
- added J1: Conn_01x06, Connector_JST:JST_SH_SM06B-SRSS-TB_1x06-1MP_P1.00mm_Horizontal, B.Cu at (152.4, 87.9)
Connections:
- IC1 pad 1: Net-(IC1-Pad1) -> /AVDD
- IC1 pad 10: Net-(IC1-Pad10) -> /SCL
- IC1 pad 11: Net-(IC1-Pad11) -> /AVDD
- IC1 pad 12: Net-(IC1-Pad12) -> GND
- IC1 pad 2: Net-(IC1-Pad2) -> GND
- IC1 pad 3: Net-(IC1-Pad3) -> GND
- IC1 pad 4: Net-(IC1-Pad4) -> GND
- IC1 pad 5: Net-(IC1-Pad5) -> /XSHUT
- IC1 pad 6: Net-(IC1-Pad6) -> GND
- IC1 pad 7: Net-(IC1-Pad7) -> /GPIO1
- IC1 pad 8: Net-(IC1-Pad8) -> (no net)
- IC1 pad 9: Net-(IC1-Pad9) -> /SDA
Routing:
- net /GPIO1: track 0.00 -> 14.3 mm, vias 0 -> 1
- net /AVDD: track 0.00 -> 9.78 mm, vias 0 -> 1
- net /XSHUT: track 0.00 -> 7.14 mm, vias 0 -> 1
- net /SDA: track 0.00 -> 5.20 mm, vias 0 -> 1
- net /SCL: track 0.00 -> 5.12 mm, vias 0 -> 1
- net GND: track 0.00 -> 3.70 mm, vias 0 -> 1
- added copper zone on F.Cu, net GND
Other:
- board outline added: 9.8 x 6.6 mm
- board text added: "RX TX"
- board text added: "VL53L1X"
